Commit message: flight controller

File: quad_description/urdf/quadrotor_base.urdf.xacro (robot description, xacro)
@@ -7,9 +7,9 @@
       <inertial>
         <mass value="1.477" />
-        <origin xyz="0 0 0.18" rpy="0 0 0"/>
+        <origin xyz="0 0 1.18" rpy="0 0 0"/>
         <inertia ixx="0.01152" ixy="0.0" ixz="0.0" iyy="0.01152" iyz="0.0" izz="0.0218" />
       </inertial>
       <visual>
-        <origin xyz="0 0 0.18" rpy="0 0 0" />
+        <origin xyz="0 0 1.18" rpy="0 0 0" />
         <geometry>
           <mesh filename="package://quad_description/meshes/quadrotor/quadrotor_base.dae"/>
@@ -17,5 +17,5 @@
       </visual>
       <collision>
-        <origin xyz="0 0 0.18" rpy="0 0 0" />
+        <origin xyz="0 0 1.18" rpy="0 0 0" />
         <geometry>
           <mesh filename="package://quad_description/meshes/quadrotor/quadrotor_base.stl"/>
